File: esp_kicad/esp_kicad.kicad_sch (KiCad schematic)
At the start: 22 parts, among them M1 Motor_Servo, M2 Motor_Servo, SW1 SW_Push, U1 L7805, U2 PIC16F1789

Commit message: Kikad updated
Parts:
- removed C4, C5: 100nF, symbol mylibrary:C
- added C4: 2200µF, symbol mylibrary:C_Polarized
- D1: value DIODE -> 1N4001
- R1, R2, R3, R4: value 330Ω -> 100Ω
Connections:
- net 0V: now also R1.2, R2.2, R3.2, R4.2, C4.2; no longer R5.2, R6.2, R7.2, R8.2
- net at C2.1, C3.1, M1.2 (+)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: now also R5.1, R6.1, R7.1, R8.1, C4.1; no longer R1.1, R2.1, R3.1, R4.1
- net at M2.1 (PWM): now also U2.16 (RC1); no longer U2.36 (RB3)
- net at R9.1: now also U2.33 (RBO); no longer U2.34 (RB1)
- net at M1.1 (PWM): now also U2.17 (RC2); no longer U2.33 (RBO)
- new net: R1.1, R5.2, U2.2 (RAO)
- new net: R2.1, R6.2, U2.3 (RA1)
- new net: R3.1, R7.2, U2.4 (RA2)
- new net: R4.1, R8.2, U2.5 (RA3)
Other:
- moved on the sheet: C1, C2, C3, D1, D2, R9, U1, U2

Commit message: Project V1.0
Parts:
- removed R10: 10kΩ, symbol mylibrary:R_US
- removed SW1: SW_Push, symbol mylibrary:SW_Push
Connections:
- net RESET: no longer names the net of U2.1 (VPP/~{MCLR}/RE3)
Changed lines of the file:
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@@
   (junction (at 50.8 99.06) (diameter 0) (color 0 0 0 0)
   )
-  (junction (at 87.63 130.81) (diameter 0) (color 0 0 0 0)
-  )
   (junction (at 237.49 99.06) (diameter 0) (color 0 0 0 0)
   )
@@
     (stroke (width 0) (type default) (color 0 0 0 0))
   )
-  (wire (pts (xy 100.33 130.81) (xy 104.14 130.81))
-    (stroke (width 0) (type default) (color 0 0 0 0))
-  )
   (wire (pts (xy 87.63 54.61) (xy 87.63 66.04))
     (stroke (width 0) (type default) (color 0 0 0 0))
@@
     (stroke (width 0) (type default) (color 0 0 0 0))
   )
-  (wire (pts (xy 207.01 31.75) (xy 213.36 31.75))
-    (stroke (width 0) (type default) (color 0 0 0 0))
-  )
   (wire (pts (xy 162.56 22.86) (xy 194.31 22.86))
     (stroke (width 0) (type default) (color 0 0 0 0))
@@
     (stroke (width 0) (type default) (color 0 0 0 0))
   )
-  (wire (pts (xy 87.63 130.81) (xy 90.17 130.81))
-    (stroke (width 0) (type default) (color 0 0 0 0))
-  )
-  (wire (pts (xy 87.63 130.81) (xy 87.63 116.84))
-    (stroke (width 0) (type default) (color 0 0 0 0))
-  )
   (wire (pts (xy 87.63 73.66) (xy 87.63 99.06))
     (stroke (width 0) (type default) (color 0 0 0 0))
@@
     (stroke (width 0) (type default) (color 0 0 0 0))
   )
-  (wire (pts (xy 69.85 130.81) (xy 76.2 130.81))
-    (stroke (width 0) (type default) (color 0 0 0 0))
-  )
-  (wire (pts (xy 213.36 31.75) (xy 213.36 35.56))
-    (stroke (width 0) (type default) (color 0 0 0 0))
-  )
   (wire (pts (xy 149.86 99.06) (xy 162.56 99.06))
     (stroke (width 0) (type default) (color 0 0 0 0))
@@
   )
   (wire (pts (xy 129.54 58.42) (xy 129.54 66.04))
-    (stroke (width 0) (type default) (color 0 0 0 0))
-  )
-  (wire (pts (xy 83.82 130.81) (xy 87.63 130.81))
     (stroke (width 0) (type default) (color 0 0 0 0))
   )
@@
     (effects (font (size 2 2) (thickness 0.254) bold) (justify left bottom))
   )
-  (global_label "RESET" (shape input) (at 87.63 116.84 90) (fields_autoplaced)
-    (effects (font (size 1.27 1.27)) (justify left))
-    (property "Intersheet References" "${INTERSHEET_REFS}" (id 0) (at 87.5506 108.6817 90)
-      (effects (font (size 1.27 1.27)) (justify left) hide)
-    )
-  )
-  (global_label "RESET" (shape input) (at 207.01 31.75 180) (fields_autoplaced)
-    (effects (font (size 1.27 1.27)) (justify right))
-    (property "Intersheet References" "${INTERSHEET_REFS}" (id 0) (at 198.8517 31.8294 0)
-      (effects (font (size 1.27 1.27)) (justify left) hide)
-    )
-  )
   (symbol (lib_id "mylibrary:+9V") (at 22.86 22.86 90) (unit 1)
     (in_bom yes) (on_board yes) (fields_autoplaced)
@@
     (pin "1")
     (pin "2")
-  )
-  (symbol (lib_id "mylibrary:Earth") (at 104.14 130.81 90) (unit 1)
-    (in_bom yes) (on_board yes) (fields_autoplaced)
-    (property "Reference" "#PWR?" (id 0) (at 110.49 130.81 0)
-      (effects (font (size 1.27 1.27)) hide)
-    )
-    (property "Value" "Earth" (id 1) (at 107.95 130.81 0)
-      (effects (font (size 1.27 1.27)) hide)
-    )
-    (property "Footprint" "" (id 2) (at 104.14 130.81 0)
-      (effects (font (size 1.27 1.27)) hide)
-    )
-    (property "Datasheet" "~" (id 3) (at 104.14 130.81 0)
-      (effects (font (size 1.27 1.27)) hide)
-    )
-    (pin "1")
   )
   (symbol (lib_id "mylibrary:L7805") (at 50.8 22.86 0) (unit 1)
@@
     (pin "1")
     (pin "2")
-  )
-  (symbol (lib_id "mylibrary:VDD") (at 69.85 130.81 90) (unit 1)
-    (in_bom yes) (on_board yes) (fields_autoplaced)
-    (property "Reference" "#PWR?" (id 0) (at 73.66 130.81 0)
-      (effects (font (size 1.27 1.27)) hide)
-    )
-    (property "Value" "VDD" (id 1) (at 64.77 130.81 0))
-    (property "Footprint" "" (id 2) (at 69.85 130.81 0)
-      (effects (font (size 1.27 1.27)) hide)
-    )
-    (property "Datasheet" "" (id 3) (at 69.85 130.81 0)
-      (effects (font (size 1.27 1.27)) hide)
-    )
-    (pin "1")
   )
   (symbol (lib_id "mylibrary:LDR03") (at 129.54 49.53 0) (unit 1)
@@
     (pin "2")
   )
-  (symbol (lib_id "mylibrary:SW_Push") (at 95.25 130.81 0) (unit 1)
-    (in_bom yes) (on_board yes) (fields_autoplaced)
-    (property "Reference" "SW1" (id 0) (at 93.9799 127 90)
-      (effects (font (size 1.27 1.27)) (justify left))
-    )
-    (property "Value" "SW_Push" (id 1) (at 96.5199 127 90)
-      (effects (font (size 1.27 1.27)) (justify left))
-    )
-    (property "Footprint" "" (id 2) (at 95.25 125.73 0)
-      (effects (font (size 1.27 1.27)) hide)
-    )
-    (property "Datasheet" "~" (id 3) (at 95.25 125.73 0)
-      (effects (font (size 1.27 1.27)) hide)
-    )
-    (pin "1")
-    (pin "2")
-  )
-  (symbol (lib_id "mylibrary:R_US") (at 80.01 130.81 90) (unit 1)
-    (in_bom yes) (on_board yes) (fields_autoplaced)
-    (property "Reference" "R10" (id 0) (at 80.01 124.46 90))
-    (property "Value" "10kΩ" (id 1) (at 80.01 127 90))
-    (property "Footprint" "" (id 2) (at 80.264 129.794 90)
-      (effects (font (size 1.27 1.27)) hide)
-    )
-    (property "Datasheet" "~" (id 3) (at 80.01 130.81 0)
-      (effects (font (size 1.27 1.27)) hide)
-    )
-    (pin "1")
-    (pin "2")
-  )
   (symbol (lib_id "mylibrary:Motor_Servo") (at 171.45 83.82 0) (unit 1)
     (in_bom yes) (on_board yes) (fields_autoplaced)
@@
       (reference "#PWR?") (unit 1) (value "+9V") (footprint "")
     )
-    (path "/556d31fc-fceb-4295-8afc-dd00216809e4"
-      (reference "#PWR?") (unit 1) (value "Earth") (footprint "")
-    )
-    (path "/9a7cd5c8-f14a-4135-9bbd-f067be0768ec"
-      (reference "#PWR?") (unit 1) (value "VDD") (footprint "")
-    )
     (path "/cc7790e2-18f0-4c52-a0b8-8af7c90bcea3"
       (reference "#PWR?") (unit 1) (value "0V") (footprint "")
@@
       (reference "R9") (unit 1) (value "330Ω") (footprint "")
     )
-    (path "/e330f112-dbf8-4c7c-9b68-db64b8dd8a90"
-      (reference "R10") (unit 1) (value "10kΩ") (footprint "")
-    )
-    (path "/df1fb14c-61a4-4634-84e9-8185e13709bb"
-      (reference "SW1") (unit 1) (value "SW_Push") (footprint "")
-    )
     (path "/5b13b165-4a62-4a6b-abb8-04669b5c4163"
